Commit message: Moving to the completely new IVK system and changing the gripper to a vacuum based version.

File: src/allardControl/urdf/block.urdf (robot description, URDF)
Before this commit: robot block, 1 links, 0 joints
Links:
- link block: geometry collision box size=0.1 0.1 0.05; visual box size=0.1 0.1 0.05

File: src/allardControl/urdf/ur10Gripper.urdf.xacro (robot description, xacro)
@@ -9,16 +9,331 @@
   /> -->
 <xacro:include filename="$(find ur_description)/urdf/ur10.urdf.xacro" />
-<xacro:include filename="$(find robotiq_2f_140_gripper_visualization)/urdf/robotiq_arg2f_140_model_macro.xacro" />
+<!-- <xacro:include filename="$(find robotiq_2f_140_gripper_visualization)/urdf/robotiq_arg2f_140_model_macro.xacro" /> -->
 <!-- create the robot + eef combo itself as a macro -->
 <xacro:macro name="ee_robot" params="prefix">
 <!-- instantiate UR5 and 2f gripper -->
   <xacro:ur10_robot prefix="${prefix}" joint_limited="false" transmission_hw_interface="$(arg transmission_hw_interface)"/>
-  <xacro:robotiq_arg2f_140 prefix="${prefix}gripper_" />
+  <!-- <xacro:robotiq_arg2f_140 prefix="${prefix}gripper_" /> -->
+ <link name="vacuum_gripper">
+      <gravity>0</gravity>
+      <visual>
+        <origin rpy="0 0 0" xyz="0 0 0"/>
+        <geometry>
+          <cylinder radius="0.005" length="0.01"/>
+        </geometry>
+        <material name="transparent">
+          <color rgba="0 0 0 0"/>
+        </material>
+      </visual>
+      <inertial>
+        <origin rpy="0 0 0" xyz="0.000000 0.000000 0.000000"/>
+        <mass value="0.0001"/>
+        <inertia ixx="1e-08" ixy="0" ixz="0" iyy="1e-08" iyz="0" izz="1e-08"/>
+      </inertial>
+    </link>
+    <joint name="gripper_joint" type="revolute">
+      <axis xyz="1 0 0" />
+      <parent link="ee_link" />
+      <child link="vacuum_gripper" />
+      <origin rpy="0 1.5708 0" xyz="0.01 0.0125 0" />
+      <limit effort="500" velocity="50" lower="0" upper="0" />
+      <dynamics damping="0.0" friction="10"/>
+    </joint>
+  <gazebo>
+      <plugin name="gazebo_ros_vacuum_gripper" filename="libgazebo_ros_vacuum_gripper.so">
+        <robotNamespace>/ur10/vacuum_gripper</robotNamespace>
+        <bodyName>vacuum_gripper</bodyName>
+        <topicName>grasping</topicName>
+	<maxForce>500</maxForce>
+        <maxDistance>0.05</maxDistance>
+        <minDistance>0.01</minDistance>
+      </plugin>
+  </gazebo>
+    <link name="vacuum_gripper1">
+      <gravity>0</gravity>
+      <visual>
+        <origin rpy="0 0 0" xyz="0 0 0"/>
+        <geometry>
+          <cylinder radius="0.005" length="0.01"/>
+        </geometry>
+        <material name="transparent">
+          <color rgba="0 0 0 0"/>
+        </material>
+      </visual>
+      <inertial>
+        <origin rpy="0 0 0" xyz="0.000000 0.000000 0.000000"/>
+        <mass value="0.0001"/>
+        <inertia ixx="1e-08" ixy="0" ixz="0" iyy="1e-08" iyz="0" izz="1e-08"/>
+      </inertial>
+    </link>
+    <joint name="gripper_joint1" type="revolute">
+      <axis xyz="1 0 0" />
+      <parent link="ee_link" />
+      <child link="vacuum_gripper1" />
+      <origin rpy="0 1.5708 0" xyz="0.01 -0.0125 0" />
+      <limit effort="500" velocity="50" lower="0" upper="0" />
+      <dynamics damping="0.0" friction="10"/>
+    </joint>
+  <gazebo>
+      <plugin name="gazebo_ros_vacuum_gripper1" filename="libgazebo_ros_vacuum_gripper.so">
+        <robotNamespace>/ur10/vacuum_gripper1</robotNamespace>
+        <bodyName>vacuum_gripper1</bodyName>
+        <topicName>grasping1</topicName>
+	<maxForce>500</maxForce>
+        <maxDistance>0.05</maxDistance>
+        <minDistance>0.01</minDistance>
+      </plugin>
+  </gazebo>
+    <link name="vacuum_gripper2">
+      <gravity>0</gravity>
+      <visual>
+        <origin rpy="0 0 0" xyz="0 0 0"/>
+        <geometry>
+          <cylinder radius="0.005" length="0.01"/>
+        </geometry>
+        <material name="transparent">
+          <color rgba="0 0 0 0"/>
+        </material>
+      </visual>
+      <inertial>
+        <origin rpy="0 0 0" xyz="0.000000 0.000000 0.000000"/>
+        <mass value="0.0001"/>
+        <inertia ixx="1e-08" ixy="0" ixz="0" iyy="1e-08" iyz="0" izz="1e-08"/>
+      </inertial>
+    </link>
+    <joint name="gripper_joint2" type="revolute">
+      <axis xyz="1 0 0" />
+      <parent link="ee_link" />
+      <child link="vacuum_gripper2" />
+      <origin rpy="0 1.5708 0" xyz="0.01 0 0.0125" />
+      <limit effort="500" velocity="50" lower="0" upper="0" />
+      <dynamics damping="0.0" friction="10"/>
+    </joint>
+  <gazebo>
+      <plugin name="gazebo_ros_vacuum_gripper2" filename="libgazebo_ros_vacuum_gripper.so">
+        <robotNamespace>/ur10/vacuum_gripper2</robotNamespace>
+        <bodyName>vacuum_gripper2</bodyName>
+        <topicName>grasping2</topicName>
+	<maxForce>500</maxForce>
+        <maxDistance>0.05</maxDistance>
+        <minDistance>0.01</minDistance>
+      </plugin>
+  </gazebo>
+    <link name="vacuum_gripper3">
+      <gravity>0</gravity>
+      <visual>
+        <origin rpy="0 0 0" xyz="0 0 0"/>
+        <geometry>
+          <cylinder radius="0.005" length="0.01"/>
+        </geometry>
+        <material name="transparent">
+          <color rgba="0 0 0 0"/>
+        </material>
+      </visual>
+      <inertial>
+        <origin rpy="0 0 0" xyz="0.000000 0.000000 0.000000"/>
+        <mass value="0.0001"/>
+        <inertia ixx="1e-08" ixy="0" ixz="0" iyy="1e-08" iyz="0" izz="1e-08"/>
+      </inertial>
+    </link>
+    <joint name="gripper_joint3" type="revolute">
+      <axis xyz="1 0 0" />
+      <parent link="ee_link" />
+      <child link="vacuum_gripper3" />
+      <origin rpy="0 1.5708 0" xyz="0.01 0 -0.0125" />
+      <limit effort="500" velocity="50" lower="0" upper="0" />
+      <dynamics damping="0.0" friction="10"/>
+    </joint>
+  <gazebo>
+      <plugin name="gazebo_ros_vacuum_gripper3" filename="libgazebo_ros_vacuum_gripper.so">
+        <robotNamespace>/ur10/vacuum_gripper3</robotNamespace>
+        <bodyName>vacuum_gripper3</bodyName>
+        <topicName>grasping2</topicName>
+	<maxForce>500</maxForce>
+        <maxDistance>0.05</maxDistance>
+        <minDistance>0.01</minDistance>
+      </plugin>
+  </gazebo>
+  <link name="vacuum_gripper4">
+    <gravity>0</gravity>
+    <visual>
+      <origin rpy="0 0 0" xyz="0 0 0"/>
+      <geometry>
+        <cylinder radius="0.005" length="0.01"/>
+      </geometry>
+      <material name="transparent">
+        <color rgba="0 0 0 0"/>
+      </material>
+    </visual>
+    <inertial>
+      <origin rpy="0 0 0" xyz="0.000000 0.000000 0.000000"/>
+      <mass value="0.0001"/>
+      <inertia ixx="1e-08" ixy="0" ixz="0" iyy="1e-08" iyz="0" izz="1e-08"/>
+    </inertial>
+  </link>
+  <joint name="gripper_joint4" type="revolute">
+    <axis xyz="1 0 0" />
+    <parent link="ee_link" />
+    <child link="vacuum_gripper4" />
+    <origin rpy="0 1.5708 0" xyz="0.01 0 0" />
+    <limit effort="500" velocity="50" lower="0" upper="0" />
+    <dynamics damping="0.0" friction="10"/>
+  </joint>
+  <gazebo>
+    <plugin name="gazebo_ros_vacuum_gripper4" filename="libgazebo_ros_vacuum_gripper.so">
+      <robotNamespace>/ur10/vacuum_gripper4</robotNamespace>
+      <bodyName>vacuum_gripper4</bodyName>
+      <topicName>grasping4</topicName>
+  <maxForce>500</maxForce>
+      <maxDistance>0.05</maxDistance>
+      <minDistance>0.01</minDistance>
+    </plugin>
+  </gazebo>
+  <link name="vacuum_gripper5">
+    <gravity>0</gravity>
+    <visual>
+      <origin rpy="0 0 0" xyz="0 0 0"/>
+      <geometry>
+        <cylinder radius="0.005" length="0.01"/>
+      </geometry>
+      <material name="transparent">
+        <color rgba="0 0 0 0"/>
+      </material>
+    </visual>
+    <inertial>
+      <origin rpy="0 0 0" xyz="0.000000 0.000000 0.000000"/>
+      <mass value="0.0001"/>
+      <inertia ixx="1e-08" ixy="0" ixz="0" iyy="1e-08" iyz="0" izz="1e-08"/>
+    </inertial>
+  </link>
+  <joint name="gripper_joint5" type="revolute">
+    <axis xyz="1 0 0" />
+    <parent link="ee_link" />
+    <child link="vacuum_gripper5" />
+    <origin rpy="0 1.5708 0" xyz="0.01 0.0125 0.0125" />
+    <limit effort="500" velocity="50" lower="0" upper="0" />
+    <dynamics damping="0.0" friction="10"/>
+  </joint>
+<gazebo>
+    <plugin name="gazebo_ros_vacuum_gripper" filename="libgazebo_ros_vacuum_gripper.so">
+      <robotNamespace>/ur10/vacuum_gripper5</robotNamespace>
+      <bodyName>vacuum_gripper5</bodyName>
+      <topicName>grasping5</topicName>
+<maxForce>500</maxForce>
+      <maxDistance>0.05</maxDistance>
+      <minDistance>0.01</minDistance>
+    </plugin>
+</gazebo>
+  <link name="vacuum_gripper6">
+    <gravity>0</gravity>
+    <visual>
+      <origin rpy="0 0 0" xyz="0 0 0"/>
+      <geometry>
+        <cylinder radius="0.005" length="0.01"/>
+      </geometry>
+      <material name="transparent">
+        <color rgba="0 0 0 0"/>
+      </material>
+    </visual>
+    <inertial>
+      <origin rpy="0 0 0" xyz="0.000000 0.000000 0.000000"/>
+      <mass value="0.0001"/>
+      <inertia ixx="1e-08" ixy="0" ixz="0" iyy="1e-08" iyz="0" izz="1e-08"/>
+    </inertial>
+  </link>
+  <joint name="gripper_joint6" type="revolute">
+    <axis xyz="1 0 0" />
+    <parent link="ee_link" />
+    <child link="vacuum_gripper6" />
+    <origin rpy="0 1.5708 0" xyz="0.01 -0.0125 0.0125" />
+    <limit effort="500" velocity="50" lower="0" upper="0" />
+    <dynamics damping="0.0" friction="10"/>
+  </joint>
+<gazebo>
+    <plugin name="gazebo_ros_vacuum_gripper1" filename="libgazebo_ros_vacuum_gripper.so">
+      <robotNamespace>/ur10/vacuum_gripper6</robotNamespace>
+      <bodyName>vacuum_gripper6</bodyName>
+      <topicName>grasping6</topicName>
+<maxForce>500</maxForce>
+      <maxDistance>0.05</maxDistance>
+      <minDistance>0.01</minDistance>
+    </plugin>
+</gazebo>
+  <link name="vacuum_gripper7">
+    <gravity>0</gravity>
+    <visual>
+      <origin rpy="0 0 0" xyz="0 0 0"/>
+      <geometry>
+        <cylinder radius="0.005" length="0.01"/>
+      </geometry>
+      <material name="transparent">
+        <color rgba="0 0 0 0"/>
+      </material>
+    </visual>
+    <inertial>
+      <origin rpy="0 0 0" xyz="0.000000 0.000000 0.000000"/>
+      <mass value="0.0001"/>
+      <inertia ixx="1e-08" ixy="0" ixz="0" iyy="1e-08" iyz="0" izz="1e-08"/>
+    </inertial>
+  </link>
+  <joint name="gripper_joint7" type="revolute">
+    <axis xyz="1 0 0" />
+    <parent link="ee_link" />
+    <child link="vacuum_gripper7" />
+    <origin rpy="0 1.5708 0" xyz="0.01 0.0125 -0.0125" />
+    <limit effort="500" velocity="50" lower="0" upper="0" />
+    <dynamics damping="0.0" friction="10"/>
+  </joint>
+<gazebo>
+    <plugin name="gazebo_ros_vacuum_gripper7" filename="libgazebo_ros_vacuum_gripper.so">
+      <robotNamespace>/ur10/vacuum_gripper7</robotNamespace>
+      <bodyName>vacuum_gripper7</bodyName>
+      <topicName>grasping7</topicName>
+<maxForce>500</maxForce>
+      <maxDistance>0.05</maxDistance>
+      <minDistance>0.01</minDistance>
+    </plugin>
+</gazebo>
+  <link name="vacuum_gripper8">
+    <gravity>0</gravity>
+    <visual>
+      <origin rpy="0 0 0" xyz="0 0 0"/>
+      <geometry>
+        <cylinder radius="0.005" length="0.01"/>
+      </geometry>
+      <material name="transparent">
+        <color rgba="0 0 0 0"/>
+      </material>
+    </visual>
+    <inertial>
+      <origin rpy="0 0 0" xyz="0.000000 0.000000 0.000000"/>
+      <mass value="0.0001"/>
+      <inertia ixx="1e-08" ixy="0" ixz="0" iyy="1e-08" iyz="0" izz="1e-08"/>
+    </inertial>
+  </link>
+  <joint name="gripper_joint8" type="revolute">
+    <axis xyz="1 0 0" />
+    <parent link="ee_link" />
+    <child link="vacuum_gripper8" />
+    <origin rpy="0 1.5708 0" xyz="0.01 -0.0125 -0.0125" />
+    <limit effort="500" velocity="50" lower="0" upper="0" />
+    <dynamics damping="0.0" friction="10"/>
+  </joint>
+<gazebo>
+    <plugin name="gazebo_ros_vacuum_gripper8" filename="libgazebo_ros_vacuum_gripper.so">
+      <robotNamespace>/ur10/vacuum_gripper8</robotNamespace>
+      <bodyName>vacuum_gripper8</bodyName>
+      <topicName>grasping8</topicName>
+<maxForce>500</maxForce>
+      <maxDistance>0.05</maxDistance>
+      <minDistance>0.01</minDistance>
+    </plugin>
+</gazebo>
   <!-- attach gripper -->
-  <joint name="${prefix}tool0-${prefix}gripper_robotiq_arg2f_base_link" type="fixed">
+  <!-- <joint name="${prefix}tool0-${prefix}gripper_base_link" type="fixed">
     <origin xyz="0 0 0" rpy="${0} ${0} ${pi}" />
     <parent link="${prefix}tool0" />
     <child link="${prefix}gripper_robotiq_arg2f_base_link" />
-  </joint>
+  </joint> -->
   <link name="world" />
   <joint name="world_joint" type="fixed">

Commit message: Updates as I move from a gripper to virtual joint hack.

File: src/allardControl/urdf/block.urdf (robot description, URDF)
Before this commit: robot block, 1 links, 0 joints
Links:
- link block: mass 0.5 -> 0.001

File: src/allardControl/urdf/ur10Gripper.urdf.xacro (robot description, xacro)
@@ -45,7 +45,7 @@
         <bodyName>vacuum_gripper</bodyName>
         <topicName>grasping</topicName>
-	<maxForce>500</maxForce>
-        <maxDistance>0.05</maxDistance>
-        <minDistance>0.01</minDistance>
+      	<maxForce>500</maxForce>
+        <maxDistance>1</maxDistance>
+        <minDistance>0.1</minDistance>
       </plugin>
   </gazebo>
@@ -80,7 +80,7 @@
         <bodyName>vacuum_gripper1</bodyName>
         <topicName>grasping1</topicName>
-	<maxForce>500</maxForce>
-        <maxDistance>0.05</maxDistance>
-        <minDistance>0.01</minDistance>
+      	<maxForce>500</maxForce>
+        <maxDistance>1</maxDistance>
+        <minDistance>0.1</minDistance>
       </plugin>
   </gazebo>
@@ -115,7 +115,7 @@
         <bodyName>vacuum_gripper2</bodyName>
         <topicName>grasping2</topicName>
-	<maxForce>500</maxForce>
-        <maxDistance>0.05</maxDistance>
-        <minDistance>0.01</minDistance>
+	      <maxForce>500</maxForce>
+        <maxDistance>1</maxDistance>
+        <minDistance>0.1</minDistance>
       </plugin>
   </gazebo>
@@ -150,7 +150,7 @@
         <bodyName>vacuum_gripper3</bodyName>
         <topicName>grasping2</topicName>
-	<maxForce>500</maxForce>
-        <maxDistance>0.05</maxDistance>
-        <minDistance>0.01</minDistance>
+	      <maxForce>500</maxForce>
+        <maxDistance>1</maxDistance>
+        <minDistance>0.1</minDistance>
       </plugin>
   </gazebo>
@@ -185,7 +185,7 @@
       <bodyName>vacuum_gripper4</bodyName>
       <topicName>grasping4</topicName>
-  <maxForce>500</maxForce>
-      <maxDistance>0.05</maxDistance>
-      <minDistance>0.01</minDistance>
+      <maxForce>500</maxForce>
+      <maxDistance>1</maxDistance>
+      <minDistance>0.1</minDistance>
     </plugin>
   </gazebo>
@@ -220,7 +220,7 @@
       <bodyName>vacuum_gripper5</bodyName>
       <topicName>grasping5</topicName>
-<maxForce>500</maxForce>
-      <maxDistance>0.05</maxDistance>
-      <minDistance>0.01</minDistance>
+      <maxForce>500</maxForce>
+      <maxDistance>1</maxDistance>
+      <minDistance>0.1</minDistance>
     </plugin>
 </gazebo>
@@ -255,7 +255,7 @@
       <bodyName>vacuum_gripper6</bodyName>
       <topicName>grasping6</topicName>
-<maxForce>500</maxForce>
-      <maxDistance>0.05</maxDistance>
-      <minDistance>0.01</minDistance>
+      <maxForce>500</maxForce>
+      <maxDistance>1</maxDistance>
+      <minDistance>0.1</minDistance>
     </plugin>
 </gazebo>
@@ -290,7 +290,7 @@
       <bodyName>vacuum_gripper7</bodyName>
       <topicName>grasping7</topicName>
-<maxForce>500</maxForce>
-      <maxDistance>0.05</maxDistance>
-      <minDistance>0.01</minDistance>
+      <maxForce>500</maxForce>
+      <maxDistance>1</maxDistance>
+      <minDistance>0.1</minDistance>
     </plugin>
 </gazebo>
@@ -325,7 +325,7 @@
       <bodyName>vacuum_gripper8</bodyName>
       <topicName>grasping8</topicName>
-<maxForce>500</maxForce>
-      <maxDistance>0.05</maxDistance>
-      <minDistance>0.01</minDistance>
+      <maxForce>500</maxForce>
+      <maxDistance>1</maxDistance>
+      <minDistance>0.1</minDistance>
     </plugin>
 </gazebo>
